File: 5th semester/Electromagnetic Measurements/Projeto/projeto_transformador_de_tensao/tension_conversor_revised2.kicad_pcb (KiCad board)
At the start: 2 copper layers, 76 parts

Commit message: Add revised board 2.0 and 3.0 to electromag measurements, and initial data for report 7 circuits lab
Parts:
- removed the ? at (118.7, 57.8)
- removed the ? at (120.0, 38.7)
- removed the ? at (113.7, 36.2)
- removed the ? at (118.7, 47.6)
- removed the ? at (111.1, 43.8)
- removed the ? at (125.1, 38.7)
- removed the ? at (113.7, 32.4)
- removed the ? at (130.8, 27.3)
- removed the ? at (114.3, 48.9)
- removed the ? at (127.0, 22.2)
- removed the ? at (113.7, 43.8)
- removed the ? at (130.8, 32.4)
- removed the ? at (113.7, 22.2)
- removed the ? at (126.4, 57.8)
- removed the ? at (130.8, 48.9)
- removed the ? at (113.7, 27.3)
- removed the ? at (114.3, 56.5)
- removed the ? at (130.8, 56.5)
- removed the ? at (126.4, 47.6)
- removed the ? at (118.7, 52.7)
- removed the ? at (126.4, 52.7)
- removed the ? at (127.0, 29.8)
- removed the ? at (130.8, 29.8)
- removed the ? at (121.3, 29.8)
- removed the REF** at (93.3, 52.1)
- removed the REF** at (98.4, 35.6)
- removed the REF** at (101.0, 43.2)
- removed the REF** at (86.4, 21.6)
- removed the REF** at (90.8, 29.2)
- removed the REF** at (85.7, 47.0)
- removed the REF** at (85.7, 52.1)
- removed the REF** at (81.3, 48.3)
- removed the REF** at (97.8, 48.3)
- removed the REF** at (85.7, 57.1)
- added ?: , , F.Cu at (152.6, 34.2)
- added ?: , , F.Cu at (129.3, 30.0)
- added ?: , , F.Cu at (152.7, 52.5)
- added ?: , , F.Cu at (145.3, 45.3)
- added ?: , , F.Cu at (141.2, 34.1)
- added ?: , , F.Cu at (146.2, 27.0)
- added ?: , , F.Cu at (152.7, 59.2)
- added ?: , , F.Cu at (146.3, 31.6)
- added ?: , , F.Cu at (145.5, 55.7)
- added ?: , , F.Cu at (129.2, 42.9)
- added ?: , , F.Cu at (137.6, 55.8)
- added ?: , , F.Cu at (136.1, 34.1)
- added ?: , , F.Cu at (129.2, 51.9)
- added ?: , , F.Cu at (129.2, 46.9)
- added ?: , , F.Cu at (152.6, 31.6)
- added ?: , , F.Cu at (129.2, 36.1)
- added ?: , , F.Cu at (129.3, 25.0)
- added ?: , , F.Cu at (137.5, 45.2)
- added ?: , , F.Cu at (146.2, 20.3)
- added ?: , , F.Cu at (129.3, 20.0)
- added ?: , , F.Cu at (137.6, 64.5)
- added ?: , , F.Cu at (145.5, 64.5)
- added ?: , , F.Cu at (152.6, 29.0)
- added ?: , , F.Cu at (129.2, 59.6)
- added REF**: Pin_D0.7mm_L6.5mm_W1.8mm_FlatFork, Connector_Pin:Pin_D0.7mm_L6.5mm_W1.8mm_FlatFork, F.Cu at (105.9, 46.5)
- added REF**: D_A-405_P7.62mm_Horizontal, Diode_THT:D_A-405_P7.62mm_Horizontal, F.Cu at (105.9, 51.5)
- added REF**: D_A-405_P7.62mm_Horizontal, Diode_THT:D_A-405_P7.62mm_Horizontal, F.Cu at (90.0, 64.2)
- added REF**: Pin_D0.7mm_L6.5mm_W1.8mm_FlatFork, Connector_Pin:Pin_D0.7mm_L6.5mm_W1.8mm_FlatFork, F.Cu at (90.0, 55.3)
- added REF**: D_A-405_P7.62mm_Horizontal, Diode_THT:D_A-405_P7.62mm_Horizontal, F.Cu at (82.4, 51.5)
- added REF**: D_A-405_P7.62mm_Horizontal, Diode_THT:D_A-405_P7.62mm_Horizontal, F.Cu at (90.0, 45.2)
- added REF**: R_Axial_DIN0204_L3.6mm_D1.6mm_P7.62mm_Horizontal, Resistor_THT:R_Axial_DIN0204_L3.6mm_D1.6mm_P7.62mm_Horizontal, F.Cu at (105.9, 35.0)
- added REF**: Pin_D0.7mm_L6.5mm_W1.8mm_FlatFork, Connector_Pin:Pin_D0.7mm_L6.5mm_W1.8mm_FlatFork, F.Cu at (97.7, 55.3)
- added REF**: R_Axial_DIN0204_L3.6mm_D1.6mm_P7.62mm_Horizontal, Resistor_THT:R_Axial_DIN0204_L3.6mm_D1.6mm_P7.62mm_Horizontal, F.Cu at (88.8, 19.8)
- added REF**: Pin_D0.7mm_L6.5mm_W1.8mm_FlatFork, Connector_Pin:Pin_D0.7mm_L6.5mm_W1.8mm_FlatFork, F.Cu at (88.8, 31.2)
- moved ? 9.16 mm to (15.2, 45.7)
- moved REF** 8.12 mm to (93.9, 33.8)
- moved REF** 7.66 mm to (105.9, 27.4)
- moved ? 7.18 mm to (21.6, 27.9)
- moved REF** 6.13 mm to (64.9, 87.4)
- moved REF** 4.95 mm to (58.5, 69.7)
- moved REF** 3.69 mm to (31.9, 64.6)
- moved REF** 3.69 mm to (16.6, 87.4)
- moved REF** 3.69 mm to (53.5, 87.4)
- moved REF** 3.69 mm to (45.8, 69.7)
- moved REF** 3.69 mm to (53.5, 77.3)
- moved REF** 3.69 mm to (20.4, 79.8)
- moved REF** 3.69 mm to (34.4, 74.7)
- moved REF** 3.69 mm to (45.8, 59.5)
- moved REF** 3.69 mm to (16.6, 64.6)
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Routing:
- net (no net): track 483.3 -> 390.4 mm
